Commit message: 10th April

File: src/ur3robot_description/urdf/ur3robot.urdf.xacro (robot description, xacro)
@@ -4,6 +4,16 @@
     <xacro:property name="effort" value="30.0"/>
     <xacro:property name="velocity" value="10.0"/>
+    <xacro:macro name="default_inertial" params="mass">
+        <inertial>
+            <mass value="${mass}"/>
+            <inertia ixx="1.0" ixy="0.0" ixz="0.0"
+                     iyy="1.0" iyz="0.0"
+                     izz="1.0">
+            </inertia>
+        </inertial>
+    </xacro:macro>
     <link name="world"/>
     <link name="base_link">
+        <xacro:default_inertial mass="1.0"/>
         <visual>
             <origin xyz="-0.5 -0.5 0" rpy="0 0 0"/>
@@ -15,4 +25,10 @@
             </material>
         </visual>
+        <collision>
+            <origin xyz="-0.5 -0.5 0" rpy="0 0 0"/>
+            <geometry>
+                <mesh filename="package://ur3robot_description/meshes/basement.STL" scale="0.01 0.01 0.01"/>
+            </geometry>
+        </collision>
     </link>
     <joint name="world_base_joint" type="fixed">
@@ -22,4 +38,5 @@
     </joint>
     <link name="base_plate">
+        <xacro:default_inertial mass="0.1"/>
         <visual>
             <origin xyz="-0.39 -0.39 -0.56"/>
@@ -31,4 +48,10 @@
             </material>
         </visual>
+        <collision>
+            <origin xyz="-0.39 -0.39 -0.56"/>
+            <geometry>
+                <mesh filename="package://ur3robot_description/meshes/base_plate.STL" scale="0.01 0.01 0.01"/>
+            </geometry>
+        </collision>
     </link>
     <joint name="base_link_base_plate_joint" type="revolute">
@@ -40,4 +63,5 @@
     </joint>
     <link name="forward_drive_arm">
+        <xacro:default_inertial mass="0.1"/>
         <visual>
             <origin xyz="0.19 0.06 -0.08" rpy="0 -${PI/2} ${PI/2}"/>
@@ -49,4 +73,10 @@
             </material>
         </visual>
+        <collision>
+            <origin xyz="0.19 0.06 -0.08" rpy="0 -${PI/2} ${PI/2}"/>
+            <geometry>
+                <mesh filename="package://ur3robot_description/meshes/forward_drive_arm.STL" scale="0.01 0.01 0.01"/>
+            </geometry>
+        </collision>
     </link>
     <joint name="base_plate_forward_drive_arm_joint" type="revolute">
@@ -58,4 +88,5 @@
     </joint>
     <link name="horizontal_arm">
+        <xacro:default_inertial mass="0.1"/>
         <visual>
             <origin xyz="-0.03 -0.4 -0.06" rpy="${PI/2} 0 ${PI/2}"/>
@@ -67,4 +98,10 @@
             </material>
         </visual>
+        <collision>
+            <origin xyz="-0.03 -0.4 -0.06" rpy="${PI/2} 0 ${PI/2}"/>
+            <geometry>
+                <mesh filename="package://ur3robot_description/meshes/horizontal_arm.STL" scale="0.01 0.01 0.01"/>
+            </geometry>
+        </collision>
     </link>
     <joint name="forward_drive_arm_horizontal_arm_joint" type="revolute">
@@ -76,4 +113,5 @@
     </joint>
     <link name="claw_support">
+        <xacro:default_inertial mass="0.05"/>
         <visual>
             <origin xyz="0 -0.05 -0.15" rpy="0 0 ${PI/2}"/>
@@ -85,4 +123,10 @@
             </material>
         </visual>
+        <collision>
+            <origin xyz="0 -0.05 -0.15" rpy="0 0 ${PI/2}"/>
+            <geometry>
+                <mesh filename="package://ur3robot_description/meshes/claw_support.STL" scale="0.01 0.01 0.01"/>
+            </geometry>
+        </collision>
     </link>
     <joint name="horizontal_arm_claw_support_joint" type="fixed">
@@ -92,4 +136,5 @@
     </joint>
     <link name="gripper_right">
+        <xacro:default_inertial mass="0.01"/>
         <visual>
             <origin xyz="-0.1 0.5 -0.1" rpy="0 0 -${PI/2}"/>
@@ -101,4 +146,10 @@
             </material>
         </visual>
+        <collision>
+            <origin xyz="-0.1 0.5 -0.1" rpy="0 0 -${PI/2}"/>
+            <geometry>
+                <mesh filename="package://ur3robot_description/meshes/right_finger.STL" scale="0.01 0.01 0.01"/>
+            </geometry>
+        </collision>
     </link>
     <joint name="claw_support_gripper_right_joint" type="revolute">
@@ -110,4 +161,5 @@
     </joint>
     <link name="gripper_left">
+        <xacro:default_inertial mass="0.01"/>
         <visual>
             <origin xyz="-0.04 0.5 -0.1" rpy="0 0 -${PI/2}"/>
@@ -119,4 +171,10 @@
             </material>
         </visual>
+        <collision>
+            <origin xyz="-0.04 0.5 -0.1" rpy="0 0 -${PI/2}"/>
+            <geometry>
+                <mesh filename="package://ur3robot_description/meshes/left_finger.STL" scale="0.01 0.01 0.01"/>
+            </geometry>
+        </collision>
     </link>
     <joint name="claw_support_gripper_left_joint" type="revolute">
